File: pcb/hedghehog-lite/hedgehog-lite.kicad_pcb (KiCad board)
At the start: 2 copper layers, 40 parts, among them J1 Conn_01x04, J2 AVR-ISP-6, K00 1u, K01 1u, K10 1u, K11 1u, SW1 Reset, SW2 HWB, U1 ATmega32U4-M, Y1 16MHz

Commit message: More edits to the schematic building v1
Parts:
- added D12: 1N4148, Diode_SMD:D_0805_2012Metric, F.Cu at (270.0, 164.3)
- added D13: 1N4148, Diode_SMD:D_0805_2012Metric, F.Cu at (233.1, 173.7)
- added D14: 1N4148, Diode_SMD:D_0805_2012Metric, F.Cu at (290.2, 158.4)
- added D15: 1N4148, Diode_SMD:D_0805_2012Metric, F.Cu at (233.1, 166.6)
- added D16: 1N4148, Diode_SMD:D_0805_2012Metric, F.Cu at (153.4, 61.9)
- added D17: 1N4148, Diode_SMD:D_0805_2012Metric, F.Cu at (139.1, 61.9)
- added D18: 1N4148, Diode_SMD:D_0805_2012Metric, F.Cu at (116.7, 61.9)
- added D2: 1N4148, Diode_SMD:D_0805_2012Metric, F.Cu at (291.5, 42.9)
- added D20: 1N4148, Diode_THT:D_DO-35_SOD27_P7.62mm_Horizontal, F.Cu at (257.9, 133.3)
- added D21: 1N4148, Diode_THT:D_DO-35_SOD27_P7.62mm_Horizontal, F.Cu at (247.4, 179.8)
- added D22: 1N4148, Diode_THT:D_DO-35_SOD27_P7.62mm_Horizontal, F.Cu at (281.9, 81.0)
- added D23: 1N4148, Diode_THT:D_DO-35_SOD27_P7.62mm_Horizontal, F.Cu at (243.8, 81.0)
- added D24: 1N4148, Diode_THT:D_DO-35_SOD27_P7.62mm_Horizontal, F.Cu at (205.7, 81.0)
- added D25: 1N4148, Diode_THT:D_DO-35_SOD27_P7.62mm_Horizontal, F.Cu at (247.4, 190.4)
- added D26: 1N4148, Diode_THT:D_DO-35_SOD27_P7.62mm_Horizontal, F.Cu at (148.6, 81.0)
- added D27: 1N4148, Diode_THT:D_DO-35_SOD27_P7.62mm_Horizontal, F.Cu at (243.8, 155.9)
- added D3: 1N4148, Diode_SMD:D_0805_2012Metric, F.Cu at (290.2, 133.3)
- added D30: 1N4148, Diode_THT:D_DO-35_SOD27_P7.62mm_Horizontal, F.Cu at (233.1, 159.5)
- added D31: 1N4148, Diode_THT:D_DO-35_SOD27_P7.62mm_Horizontal, F.Cu at (243.8, 159.5)
- added D32: 1N4148, Diode_THT:D_DO-35_SOD27_P7.62mm_Horizontal, F.Cu at (233.1, 170.2)
- added D32: 1N4148, Diode_THT:D_DO-35_SOD27_P7.62mm_Horizontal, F.Cu at (277.2, 100.0)
- added D33: 1N4148, Diode_THT:D_DO-35_SOD27_P7.62mm_Horizontal, F.Cu at (225.6, 133.3)
- added D34: 1N4148, Diode_THT:D_DO-35_SOD27_P7.62mm_Horizontal, F.Cu at (233.1, 152.4)
- added D35: 1N4148, Diode_THT:D_DO-35_SOD27_P7.62mm_Horizontal, F.Cu at (162.9, 100.0)
- added D36: 1N4148, Diode_THT:D_DO-35_SOD27_P7.62mm_Horizontal, F.Cu at (258.1, 186.9)
- added D38: 1N4148, Diode_THT:D_DO-35_SOD27_P7.62mm_Horizontal, F.Cu at (279.4, 133.3)
- added D4: 1N4148, Diode_SMD:D_0805_2012Metric, F.Cu at (215.3, 42.9)
- added D40: 1N4148, Diode_THT:D_DO-35_SOD27_P7.62mm_Horizontal, F.Cu at (352.4, 72.4)
- added D41: 1N4148, Diode_THT:D_DO-35_SOD27_P7.62mm_Horizontal, F.Cu at (308.1, 116.7)
- added D42: 1N4148, Diode_THT:D_DO-35_SOD27_P7.62mm_Horizontal, F.Cu at (258.1, 183.3)
- added D43: 1N4148, Diode_THT:D_DO-35_SOD27_P7.62mm_Horizontal, F.Cu at (269.1, 113.3)
- added D44: 1N4148, Diode_THT:D_DO-35_SOD27_P7.62mm_Horizontal, F.Cu at (243.8, 163.1)
- added D45: 1N4148, Diode_THT:D_DO-35_SOD27_P7.62mm_Horizontal, F.Cu at (233.1, 155.9)
- added D46: 1N4148, Diode_THT:D_DO-35_SOD27_P7.62mm_Horizontal, F.Cu at (172.4, 116.7)
- added D5: 1N4148, Diode_SMD:D_0805_2012Metric, F.Cu at (177.2, 42.9)
- added D50: 1N4148, Diode_THT:D_DO-35_SOD27_P7.62mm_Horizontal, F.Cu at (339.1, 81.0)
- added D51: 1N4148, Diode_THT:D_DO-35_SOD27_P7.62mm_Horizontal, F.Cu at (233.1, 163.1)
- added D52: 1N4148, Diode_THT:D_DO-35_SOD27_P7.62mm_Horizontal, F.Cu at (269.1, 101.4)
- added D53: 1N4148, Diode_THT:D_DO-35_SOD27_P7.62mm_Horizontal, F.Cu at (226.4, 126.6)
- added D54: 1N4148, Diode_THT:D_DO-35_SOD27_P7.62mm_Horizontal, F.Cu at (301.0, 151.3)
- added D59: 1N4148, Diode_THT:D_DO-35_SOD27_P7.62mm_Horizontal, F.Cu at (258.1, 176.2)
- added D6: 1N4148, Diode_SMD:D_0805_2012Metric, F.Cu at (158.1, 42.9)
- added D60: 1N4148, Diode_THT:D_DO-35_SOD27_P7.62mm_Horizontal, F.Cu at (258.1, 179.8)
- added D60: 1N4148, Diode_THT:D_DO-35_SOD27_P7.62mm_Horizontal, F.Cu at (343.9, 61.9)
- added D61: 1N4148, Diode_THT:D_DO-35_SOD27_P7.62mm_Horizontal, F.Cu at (280.8, 171.4)
- added D61: 1N4148, Diode_THT:D_DO-35_SOD27_P7.62mm_Horizontal, F.Cu at (247.4, 186.9)
- added D62: 1N4148, Diode_THT:D_DO-35_SOD27_P7.62mm_Horizontal, F.Cu at (280.8, 164.3)
- added D62: 1N4148, Diode_THT:D_DO-35_SOD27_P7.62mm_Horizontal, F.Cu at (262.9, 81.0)
- added D63: 1N4148, Diode_THT:D_DO-35_SOD27_P7.62mm_Horizontal, F.Cu at (224.8, 81.0)
- added D64: 1N4148, Diode_THT:D_DO-35_SOD27_P7.62mm_Horizontal, F.Cu at (270.0, 171.4)
- added D65: 1N4148, Diode_THT:D_DO-35_SOD27_P7.62mm_Horizontal, F.Cu at (247.1, 133.3)
- added D66: 1N4148, Diode_THT:D_DO-35_SOD27_P7.62mm_Horizontal, F.Cu at (280.8, 167.9)
- added D67: 1N4148, Diode_THT:D_DO-35_SOD27_P7.62mm_Horizontal, F.Cu at (243.8, 152.4)
- added D7: 1N4148, Diode_SMD:D_0805_2012Metric, F.Cu at (214.8, 133.3)
- added D70: 1N4148, Diode_SMD:D_0805_2012Metric, F.Cu at (344.8, 41.7)
- added D71: 1N4148, Diode_THT:D_DO-35_SOD27_P7.62mm_Horizontal, F.Cu at (305.8, 61.9)
- added D71: 1N4148, Diode_THT:D_DO-35_SOD27_P7.62mm_Horizontal, F.Cu at (247.4, 176.2)
- added D72: 1N4148, Diode_THT:D_DO-35_SOD27_P7.62mm_Horizontal, F.Cu at (301.0, 133.3)
- added D72: 1N4148, Diode_THT:D_DO-35_SOD27_P7.62mm_Horizontal, F.Cu at (301.0, 154.8)
- added D73: 1N4148, Diode_THT:D_DO-35_SOD27_P7.62mm_Horizontal, F.Cu at (270.0, 167.9)
- added D73: 1N4148, Diode_THT:D_DO-35_SOD27_P7.62mm_Horizontal, F.Cu at (268.7, 133.3)
- added D74: 1N4148, Diode_THT:D_DO-35_SOD27_P7.62mm_Horizontal, F.Cu at (290.2, 154.8)
- added D74: 1N4148, Diode_THT:D_DO-35_SOD27_P7.62mm_Horizontal, F.Cu at (191.5, 61.9)
- added D78: 1N4148, Diode_THT:D_DO-35_SOD27_P7.62mm_Horizontal, F.Cu at (236.4, 133.3)
- added D79: 1N4148, Diode_THT:D_DO-35_SOD27_P7.62mm_Horizontal, F.Cu at (311.8, 133.3)
- added D8: 1N4148, Diode_SMD:D_0805_2012Metric, F.Cu at (110.5, 42.9)
- added D81: 1N4148, Diode_SMD:D_0805_2012Metric, F.Cu at (306.7, 41.7)
- added D82: 1N4148, Diode_THT:D_DO-35_SOD27_P7.62mm_Horizontal, F.Cu at (272.4, 42.9)
- added D83: 1N4148, Diode_THT:D_DO-35_SOD27_P7.62mm_Horizontal, F.Cu at (234.3, 42.9)
- added D84: 1N4148, Diode_THT:D_DO-35_SOD27_P7.62mm_Horizontal, F.Cu at (247.4, 183.3)
- added D88: 1N4148, Diode_THT:D_DO-35_SOD27_P7.62mm_Horizontal, F.Cu at (86.7, 42.9)
- added K12: 1u, acheron:MX100H, F.Cu at (290.5, 52.4)
- added K13: 1u, acheron:MX100H, F.Cu at (252.4, 52.4)
- added K14: 1u, acheron:MX100H, F.Cu at (214.3, 52.4)
- added K15: 1u, acheron:MX100H, F.Cu at (176.2, 52.4)
- added K16: 1u, acheron:MX100H, F.Cu at (157.2, 52.4)
- added K17: 1u, acheron:MX100H, F.Cu at (138.1, 52.4)
- added K18: 1.5u, acheron:MX150H, F.Cu at (114.3, 52.4)
- added K2: 1u, acheron:MX100H, F.Cu at (295.3, 33.3)
- added K20: 1u, acheron:MX100H, F.Cu at (361.9, 71.4)
- added K21: 1u, acheron:MX100H, F.Cu at (323.9, 71.4)
- added K22: 1u, acheron:MX100H, F.Cu at (285.8, 71.4)
- added K23: 1u, acheron:MX100H, F.Cu at (247.7, 71.4)
- added K24: 1u, acheron:MX100H, F.Cu at (209.6, 71.4)
- added K25: 1u, acheron:MX100H, F.Cu at (171.4, 71.4)
- added K26: 1u, acheron:MX100H, F.Cu at (152.4, 71.4)
- added K27: 2.25u, acheron:MX225H, F.Cu at (121.4, 71.4)
- added K3: 1u, acheron:MX100H, F.Cu at (257.2, 33.3)
- added K30: 1u, acheron:MX100H, F.Cu at (357.2, 90.5)
- added K31: 1u, acheron:MX100H, F.Cu at (319.1, 90.5)
- added K32: 1u, acheron:MX100H, F.Cu at (281.0, 90.5)
- added K33: 1u, acheron:MX100H, F.Cu at (242.9, 90.5)
- added K34: 1u, acheron:MX100H, F.Cu at (204.8, 90.5)
- added K35: 1u, acheron:MX100H, F.Cu at (166.7, 90.5)
- added K36: 2.75u, acheron:MX275H, F.Cu at (131.0, 90.5)
- added K38: 1u, acheron:MX100H, F.Cu at (90.5, 52.4)
- added K4: 1u, acheron:MX100H, F.Cu at (219.1, 33.3)
- added K40: 1u, acheron:MX100H, F.Cu at (338.1, 90.5)
- added K41: 1.25u, acheron:MX125H, F.Cu at (311.9, 109.5)
- added K42: 1.25u, acheron:MX125H, F.Cu at (288.1, 109.5)
- added K43: 2.75u, acheron:MX275HR, F.Cu at (250.0, 109.5)
- added K44: 1u, acheron:MX100H, F.Cu at (214.3, 109.5)
- added K45: 1u, acheron:MX100H, F.Cu at (195.3, 109.5)
- added K46: 1u, acheron:MX100H, F.Cu at (176.2, 109.5)
- added K5: 1u, acheron:MX100H, F.Cu at (181.0, 33.3)
- added K50: 1u, acheron:MX100H, F.Cu at (342.9, 71.4)
- added K51: 1u, acheron:MX100H, F.Cu at (300.0, 90.5)
- added K52: 1u, acheron:MX100H, F.Cu at (261.9, 90.5)
- added K53: 1u, acheron:MX100H, F.Cu at (223.8, 90.5)
- added K54: 1u, acheron:MX100H, F.Cu at (185.7, 90.5)
- added K6: 1u, acheron:MX100H, F.Cu at (161.9, 33.3)
- added K60: 1u, acheron:MX100H, F.Cu at (347.7, 52.4)
- added K61: 1u, acheron:MX100H, F.Cu at (304.8, 71.4)
- added K62: 1u, acheron:MX100H, F.Cu at (266.7, 71.4)
- added K63: 1u, acheron:MX100H, F.Cu at (228.6, 71.4)
- added K64: 1u, acheron:MX100H, F.Cu at (190.5, 71.4)
- added K7: 1u, acheron:MX100H, F.Cu at (142.9, 33.3)
- added K70: 1u, acheron:MX100H, F.Cu at (352.4, 33.3)
- added K71: 1u, acheron:MX100H, F.Cu at (309.6, 52.4)
- added K72: 1u, acheron:MX100H, F.Cu at (271.5, 52.4)
- added K73: 1u, acheron:MX100H, F.Cu at (233.4, 52.4)
- added K74: 1u, acheron:MX100H, F.Cu at (195.3, 52.4)
- added K8: 2u, acheron:MX200H, F.Cu at (114.3, 33.3)
- added K81: 1u, acheron:MX100H, F.Cu at (314.3, 33.3)
- added K82: 1u, acheron:MX100H, F.Cu at (276.2, 33.3)
- added K83: 1u, acheron:MX100H, F.Cu at (238.1, 33.3)
- added K84: 1u, acheron:MX100H, F.Cu at (200.0, 33.3)
- added K88: 1u, acheron:MX100H, F.Cu at (85.7, 33.3)
- D0: renamed from D1; footprint Diode_THT:D_DO-35_SOD27_P7.62mm_Horizontal -> Diode_SMD:D_SOD-123F
- D1: renamed from D3; footprint Diode_THT:D_DO-35_SOD27_P7.62mm_Horizontal -> Diode_SMD:D_0805_2012Metric
- D10: renamed from D2; footprint Diode_THT:D_DO-35_SOD27_P7.62mm_Horizontal -> Diode_SMD:D_0805_2012Metric
- D11: renamed from D4; footprint Diode_THT:D_DO-35_SOD27_P7.62mm_Horizontal -> Diode_SMD:D_0805_2012Metric
- moved K0 147.2 mm to (371.5, 33.3)
- moved D10 144.8 mm to (365.3, 61.9)
- moved D0 144.1 mm to (364.4, 41.7)
- moved K10 142.5 mm to (366.7, 52.4)
- moved K1 128.4 mm to (333.4, 33.3)
- moved D1 124.9 mm to (325.8, 41.7)
- moved D11 123.8 mm to (324.8, 61.9)
- moved K11 123.8 mm to (328.6, 52.4)
- moved U1 101.0 mm to (228.9, 112.3)
- moved C5 100.8 mm to (228.7, 105.8)
- moved C6 100.8 mm to (228.7, 99.4)
- moved Y1 100.8 mm to (228.7, 102.6)
- moved DL10 36.3 mm to (126.2, 203.5)
- moved DL11 36.3 mm to (109.4, 203.5)
- moved DL12 36.3 mm to (92.5, 203.5)
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- renumbered K00 to K0, K01 to K1
Routing:
- net COL0: track 0.00 -> 123.0 mm

Commit message: Placed all components on PCB
Parts:
- removed the D32 at (233.1, 170.2)
- removed D59, D65, D66, D67, D78, D79: 1N4148, Diode_THT:D_DO-35_SOD27_P7.62mm_Horizontal
- removed the D60 at (343.9, 61.9)
- removed the D61 at (247.4, 186.9)
- removed the D62 at (280.8, 164.3)
- removed the D71 at (247.4, 176.2)
- removed the D72 at (301.0, 133.3)
- removed the D73 at (268.7, 133.3)
- removed the D74 at (290.2, 154.8)
- removed the R2 at (151.9, 201.6)
- D0: value 1N4148 -> SM4007
- D1, D10, D11, D12, D13, D14, D15, D16, D17, D18, D2, D3, D4, D5, D6, D7, D70, D8, D81: value 1N4148 -> SM4007; footprint Diode_SMD:D_0805_2012Metric -> Diode_SMD:D_SOD-123F
- D20, D21, D22, D23, D24, D25, D26, D27, D30, D31, D32, D33, D34, D35, D36, D38, D40, D41, D42, D43, D44, D45, D46, D50, D51, D52, D53, D54, D60, D61, D62, D63, D64, D71, D72, D73, D74, D82, D83, D84, D88: value 1N4148 -> SM4007; footprint Diode_THT:D_DO-35_SOD27_P7.62mm_Horizontal -> Diode_SMD:D_SOD-123F
- SW1: moved to B.Cu
- SW2: value HWB -> SSSS811101; footprint Button_Switch_SMD:SW_DIP_SPSTx01_Slide_6.7x4.1mm_W8.61mm_P2.54mm_LowProfile -> SSSS811101:SSSS811101
- moved DL8 253.4 mm to (344.4, 90.1)
- moved DL7 238.3 mm to (324.4, 127.1)
- moved DL9 216.5 mm to (306.4, 90.1)
- moved DL6 204.4 mm to (279.4, 127.1)
- moved D38 200.6 mm to (80.9, 104.7), turned to 90 degrees
- moved DL10 181.8 mm to (268.4, 90.1)
- moved DL11 165.5 mm to (229.8, 90.1)
- moved DL12 150.7 mm to (191.8, 90.1)
- moved U1 148.8 mm to (83.8, 145.6)
- moved C5 148.5 mm to (83.8, 138.1)
- moved C6 148.4 mm to (83.8, 131.5)
- moved Y1 148.4 mm to (83.8, 134.8)
- moved DL4 142.6 mm to (234.3, 148.1)
- moved DL5 140.5 mm to (234.3, 127.1)
- moved D54 140.0 mm to (161.0, 147.6)
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- renumbered J2 to ISP
Routing:
- net COL0: track 123.0 -> 0.00 mm
Other:
- board outline added: 303 x 94 mm

Commit message: Moved pin header to allow left side conn
Parts:
- moved J1 186.3 mm to (259.0, 108.5)
- moved D22 18.9 mm to (264.0, 125.5)
- moved D12 15.3 mm to (280.5, 104.1), turned to 90 degrees
- moved D71 3.74 mm to (287.5, 107.0)
Changed lines of the file:
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@@
   )
   (footprint "random-keyboard-parts:JST-SR-4" (layer "F.Cu")
-    (at 72.884 116.3725 90)
+    (at 259 108.5 90)
     (property "LCSC Part #" "C160404")
     (property "Sheetfile" "hedgehog-lite.kicad_sch")
@@
   )
   (footprint "Diode_SMD:D_SOD-123F" (layer "F.Cu")
-    (at 277.498 112.3085 180)
+    (at 264 125.5 180)
     (descr "D_SOD-123F")
     (tags "D_SOD-123F")
@@
   )
   (footprint "Diode_SMD:D_SOD-123F" (layer "F.Cu")
-    (at 284.737 109.5145)
+    (at 287.5 107)
     (descr "D_SOD-123F")
     (tags "D_SOD-123F")
@@
   )
   (footprint "Diode_SMD:D_SOD-123F" (layer "F.Cu")
-    (at 265.814 108.3715)
+    (at 280.5 104.1 90)
     (descr "D_SOD-123F")
     (tags "D_SOD-123F")
@@
     (property "Sheetname" "Switch Matrix")
     (attr smd)
-    (fp_text reference "D12" (at -0.127 -1.905) (layer "F.SilkS")
+    (fp_text reference "D12" (at -0.127 -1.905 90) (layer "F.SilkS")
       (effects (font (size 1 1) (thickness 0.15)))
     )
-    (fp_text value "SM4007" (at 0 2.1) (layer "F.Fab")
+    (fp_text value "SM4007" (at 0 2.1 90) (layer "F.Fab")
       (effects (font (size 1 1) (thickness 0.15)))
     )
-    (fp_text user "${REFERENCE}" (at -0.127 -1.905) (layer "F.Fab")
+    (fp_text user "${REFERENCE}" (at -0.127 -1.905 90) (layer "F.Fab")
       (effects (font (size 1 1) (thickness 0.15)))
     )
@@
     (fp_line (start -0.75 0) (end -0.35 0) (layer "F.Fab") (width 0.1))
     (fp_line (start -0.35 0) (end -0.35 -0.55) (layer "F.Fab") (width 0.1))
-    (pad "1" smd rect (at -1.4 0) (size 1.1 1.1) (layers "F.Cu" "F.Paste" "F.Mask")
+    (pad "1" smd rect (at -1.4 0 90) (size 1.1 1.1) (layers "F.Cu" "F.Paste" "F.Mask")
       (net 38 "ROW1") (pinfunction "K") (pintype "passive"))
-    (pad "2" smd rect (at 1.4 0) (size 1.1 1.1) (layers "F.Cu" "F.Paste" "F.Mask")
+    (pad "2" smd rect (at 1.4 0 90) (size 1.1 1.1) (layers "F.Cu" "F.Paste" "F.Mask")
       (net 65 "Net-(D12-Pad2)") (pinfunction "A") (pintype "passive"))
     (model "${KICAD6_3DMODEL_DIR}/Diode_SMD.3dshapes/D_SOD-123F.wrl"

Commit message: Cleanup, better placement, ready to wire
Parts:
- removed ISP: AVR-ISP-6, Connector_PinHeader_1.27mm:PinHeader_2x03_P1.27mm_Vertical
- added J2: AVR-ISP-6, Connector_PinHeader_1.27mm:PinHeader_2x03_P1.27mm_Vertical, F.Cu at (62.2, 104.6)
- R2: value 10k -> 1k
- moved D46 11.0 mm to (167.4, 161.2), turned to 180 degrees
- moved D17 9.24 mm to (106.0, 104.0)
- moved D14 6.22 mm to (187.0, 104.0)
- moved D72 6.17 mm to (244.0, 104.0)
- moved D15 6.11 mm to (149.0, 104.0)
- moved D16 6.11 mm to (130.0, 104.0)
- moved D13 6.09 mm to (225.0, 104.0)
- moved D73 6.07 mm to (206.0, 104.0)
- moved D74 6.03 mm to (168.0, 104.0)
- moved JP1 4.96 mm to (80.2, 119.8)
- moved C2 4.96 mm to (77.2, 128.9)
- moved C3 4.96 mm to (77.2, 131.3)
- moved C4 4.96 mm to (77.2, 133.7)
- moved C6 4.96 mm to (82.9, 126.6)
- moved C7 4.96 mm to (90.1, 141.0)
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Other:
- board size 303 x 94 mm -> 303.6 x 95 mm

Commit message: Wiring up all parts, excluding matrix
Parts:
- moved JP1 19.6 mm to (93.6, 134.0)
- moved C6 18.7 mm to (77.0, 144.4), turned to 0 degrees
- moved D36 17.6 mm to (117.5, 144.8)
- moved C7 13.9 mm to (84.7, 128.2), turned to 180 degrees
- moved Y1 12.4 mm to (77.0, 140.8), turned to 90 degrees
- moved C5 7.09 mm to (77.0, 137.2), turned to 180 degrees
- moved R1 6.71 mm to (253.6, 158.6)
- moved D81 4.20 mm to (290.4, 86.6)
- moved D82 4.07 mm to (254.4, 87.5)
- moved C3 3.43 mm to (80.5, 130.6)
- moved C1 3.43 mm to (80.5, 125.8)
- moved C2 3.43 mm to (80.5, 128.2)
- moved C4 3.43 mm to (80.5, 133.0)
- moved D84 3.35 mm to (175.1, 87.2)
- moved D25 3.05 mm to (154.1, 128.6)
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Connections:
- DL10 pad 1: +5V -> LED_PWR_P
- DL11 pad 1: +5V -> LED_PWR_P
- DL12 pad 1: +5V -> LED_PWR_P
- DL13 pad 1: +5V -> LED_PWR_P
- DL14 pad 1: +5V -> LED_PWR_P
- DL15 pad 1: +5V -> LED_PWR_P
- DL8 pad 1: +5V -> LED_PWR_P
- DL9 pad 1: +5V -> LED_PWR_P
- U1 pad 41: unconnected-(U1-Pad41) -> RGB
Routing:
- net GND: track 0.00 -> 728.7 mm, vias 0 -> 22
- net LED_PWR_P: track 0.00 -> 600.3 mm, vias 0 -> 6
- net +5V: track 0.00 -> 491.8 mm, vias 0 -> 11
- net RST: track 0.00 -> 265.8 mm, vias 0 -> 4
- net DP: track 0.00 -> 200.9 mm, vias 0 -> 2
- net DN: track 0.00 -> 198.8 mm, vias 0 -> 2
- net COL0: track 0.00 -> 145.6 mm, vias 0 -> 6
- net Net-(DL7-Pad2): track 0.00 -> 74.1 mm, vias 0 -> 2
- net Net-(DL3-Pad2): track 0.00 -> 65.8 mm, vias 0 -> 2
- net Net-(SW2-Pad1): track 0.00 -> 64.3 mm, vias 0 -> 4
- net SCK: track 0.00 -> 54.8 mm, vias 0 -> 2
- net MISO: track 0.00 -> 54.2 mm, vias 0 -> 2
- net MOSI: track 0.00 -> 49.2 mm, vias 0 -> 1
- net Net-(DL1-Pad2): track 0.00 -> 41.6 mm
- net Net-(DL6-Pad2): track 0.00 -> 41.4 mm
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- added copper zone on F.Cu, net GND

Commit message: Added edge cuts
Parts:
- moved D6 23.1 mm to (153.8, 74.5), turned to 180 degrees
- moved D64 21.8 mm to (180.0, 112.0), turned to 180 degrees
- moved D42 20.4 mm to (279.5, 159.4), turned to 180 degrees
- moved D23 19.1 mm to (237.4, 112.1), turned to 180 degrees
- moved D43 19.1 mm to (236.6, 161.4)
- moved D26 18.1 mm to (142.0, 112.1)
- moved D34 17.9 mm to (196.7, 141.2)
- moved D25 17.8 mm to (160.9, 112.1)
- moved D54 17.7 mm to (177.5, 141.2), turned to 180 degrees
- moved D22 17.3 mm to (275.2, 112.3)
- moved D45 16.3 mm to (182.0, 161.8)
- moved D44 16.2 mm to (201.0, 161.8)
- moved D53 13.5 mm to (212.0, 143.0)
- moved D32 13.3 mm to (268.9, 143.1), turned to 90 degrees
- moved D31 12.9 mm to (306.8, 143.5), turned to 90 degrees
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Routing:
- net GND: track 728.7 -> 798.4 mm, vias 22 -> 21
- net Net-(DL10-Pad4): track 35.0 -> 3.00 mm
- net Net-(D40-Pad2): track 27.5 -> 16.4 mm, vias 2 -> 0
- net +5V: track 491.8 -> 481.4 mm
- net LED_PWR_P: track 600.3 -> 596.3 mm
- net Net-(DL3-Pad2): track 65.8 -> 68.2 mm, vias 2 -> 4
- net Net-(DL12-Pad2): track 34.9 -> 36.5 mm
- net Net-(DL13-Pad2): track 34.4 -> 35.2 mm
- net RST: track 265.8 -> 265.5 mm, vias 4 -> 3
Other:
- outline, holes or cut-outs redrawn

Commit message: all done but switches
Parts:
- added R3: 22, Resistor_SMD:R_0805_2012Metric, F.Cu at (72.6, 114.7)
- added R4: 22, Resistor_SMD:R_0805_2012Metric, F.Cu at (73.7, 118.9)
- moved D31 11.4 mm to (295.9, 146.8)
- moved D34 11.4 mm to (185.8, 144.5)
- moved D35 11.4 mm to (131.1, 150.9)
- moved D41 11.4 mm to (274.2, 162.7)
- moved D42 11.4 mm to (268.6, 162.7)
- moved K41 11.4 mm to (283.4, 161.9)
- moved K42 11.4 mm to (259.6, 161.9)
- moved K45 11.4 mm to (166.7, 161.9)
- moved K46 11.4 mm to (147.6, 161.9)
- moved SW1 11.4 mm to (242.6, 161.9)
- moved D0 11.4 mm to (346.9, 90.9)
- moved D1 11.4 mm to (306.4, 90.9)
- moved D10 11.4 mm to (331.1, 112.8)
- moved D11 11.4 mm to (293.0, 112.8)
- moved D12 11.4 mm to (269.6, 107.4)
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Connections:
- U1 pad 3: DN -> Net-(R4-Pad1)
- U1 pad 4: DP -> Net-(R3-Pad1)
Routing:
- net DP: track 200.9 -> 172.7 mm, vias 2 -> 1
- net Net-(R3-Pad1): track 0.00 -> 26.3 mm, vias 0 -> 2
- net DN: track 198.8 -> 175.0 mm, vias 2 -> 1
- net Net-(R4-Pad1): track 0.00 -> 21.9 mm, vias 0 -> 2
- net +5V: track 481.4 -> 481.3 mm, vias 11 -> 13
- removed copper zone on F.Cu, net GND
Other:
- outline, holes or cut-outs redrawn

Commit message: Columns wired up
Parts:
- moved D6 14.4 mm to (148.7, 91.0)
- moved D8 13.1 mm to (97.4, 86.3), turned to 180 degrees
Routing:
- net COL4: track 0.00 -> 342.6 mm, vias 0 -> 15
- net COL3: track 0.00 -> 310.5 mm, vias 0 -> 11
- net COL2: track 0.00 -> 239.9 mm, vias 0 -> 13
- net COL1: track 20.6 -> 221.8 mm, vias 0 -> 9
- net COL5: track 0.00 -> 185.8 mm, vias 0 -> 10
- net COL6: track 0.00 -> 154.7 mm, vias 0 -> 9
- net COL8: track 0.00 -> 75.0 mm, vias 0 -> 2
- net COL7: track 0.00 -> 55.5 mm, vias 0 -> 4
- net +5V: track 481.3 -> 483.2 mm
- net RST: track 265.5 -> 266.1 mm
