File: pcb/hedghehog-lite/hedgehog-lite.kicad_pcb (KiCad board)
At the start: 2 copper layers, 303.6 x 95 mm, 155 parts, among them J1 Conn_01x04, J2 AVR-ISP-6, K0 1u, K1 1u, K10 1u, K11 1u, K12 1u, K13 1u, K14 1u, K15 1u, K16 1u, K17 1u, K18 1.5u, K2 1u, K20 1u, K21 1u, K22 1u, K23 1u, K24 1u, K25 1u, K26 1u, K27 2.25u, K3 1u, K30 1u, K31 1u, K32 1u, K33 1u, K34 1u, K35 1u, K36 2.75u, K38 1u, K4 1u, K40 1u, K41 1.25u, K42 1.25u, K43 2.75u, K44 1u, K45 1u, K46 1u, K5 1u, K50 1u, K51 1u, K52 1u, K53 1u, K54 1u, K6 1u, K60 1u, K61 1u, K62 1u, K63 1u, K64 1u, K7 1u, K70 1u, K71 1u, K72 1u, K73 1u, K74 1u, K8 2u, K81 1u, K82 1u, K83 1u, K84 1u, K88 1u, SW1 Reset, SW2 SSSS811101, U1 ATmega32U4-M, Y1 16MHz

Commit message: Top Row done
Parts:
- moved D83 18.1 mm to (219.9, 84.3), turned to 90 degrees
- moved D82 16.1 mm to (258.0, 83.9), turned to 90 degrees
- moved D81 7.43 mm to (286.9, 90.2)
- moved D84 7.32 mm to (171.5, 90.8), turned to 180 degrees
- moved D18 6.02 mm to (100.9, 107.4)
- moved D2 3.72 mm to (273.9, 87.8), turned to 180 degrees
- moved D1 3.64 mm to (309.3, 88.6)
- moved D70 2.59 mm to (317.0, 88.5)
- moved D17 0.32 mm to (95.4, 107.4), turned to 180 degrees
Connections:
- D0 pad 1: ROW0 -> MISO
- D1 pad 1: ROW0 -> MISO
- D2 pad 1: ROW0 -> MISO
- D3 pad 1: ROW0 -> MISO
- D4 pad 1: ROW0 -> MISO
- D5 pad 1: ROW0 -> MISO
- D6 pad 1: ROW0 -> MISO
- D7 pad 1: ROW0 -> MISO
- D8 pad 1: ROW0 -> MISO
- D81 pad 1: ROW8 -> SCK
- D82 pad 1: ROW8 -> SCK
- D83 pad 1: ROW8 -> SCK
- D84 pad 1: ROW8 -> SCK
- D88 pad 1: ROW8 -> SCK
Routing:
- net MISO: track 54.2 -> 408.6 mm, vias 2 -> 13
- net SCK: track 54.8 -> 358.1 mm, vias 2 -> 13
- net Net-(D88-Pad2): track 0.00 -> 18.8 mm
- net Net-(D84-Pad2): track 0.00 -> 17.8 mm, vias 0 -> 2
- net Net-(D5-Pad2): track 0.00 -> 12.2 mm, vias 0 -> 2
- net Net-(D81-Pad2): track 0.00 -> 12.0 mm, vias 0 -> 2
- net Net-(D6-Pad2): track 0.00 -> 11.7 mm, vias 0 -> 2
- net Net-(D4-Pad2): track 0.00 -> 11.6 mm, vias 0 -> 2
- net Net-(D70-Pad2): track 25.4 -> 17.7 mm, vias 2 -> 0
- net Net-(D1-Pad2): track 0.00 -> 6.06 mm
- net Net-(D8-Pad2): track 0.00 -> 5.63 mm
- net Net-(D7-Pad2): track 0.00 -> 4.83 mm
- net Net-(D82-Pad2): track 0.00 -> 3.28 mm
- net Net-(D83-Pad2): track 0.00 -> 3.07 mm
- net LED_PWR_P: track 596.3 -> 595.2 mm
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
Commit message: All routing done
Parts:
- moved D17 18.5 mm to (113.8, 108.7), turned to 0 degrees
- moved D74 14.0 mm to (171.1, 107.3), turned to 180 degrees
- moved D60 12.4 mm to (323.2, 107.6)
- moved D21 11.3 mm to (299.5, 126.5), turned to 180 degrees
- moved D63 10.6 mm to (207.3, 126.1), turned to 180 degrees
- moved D34 6.36 mm to (180.6, 148.2)
- moved D14 5.86 mm to (181.7, 108.8)
- moved D15 5.86 mm to (143.8, 108.7)
- moved D18 5.82 mm to (95.2, 108.7), turned to 180 degrees
- moved D13 5.59 mm to (219.5, 108.8)
- moved D72 5.56 mm to (238.6, 107.4)
- moved D16 5.35 mm to (124.2, 108.8)
- moved D71 2.93 mm to (274.7, 108.1)
- moved D31 1.71 mm to (294.8, 145.5), turned to 180 degrees
- moved D61 1.64 mm to (280.7, 126.6), turned to 180 degrees
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Connections:
- K0 pad 1: COL0 -> MOSI
- K10 pad 1: COL0 -> MOSI
- K20 pad 1: COL0 -> MOSI
- K30 pad 1: COL0 -> MOSI
- K40 pad 1: COL0 -> MOSI
- K50 pad 1: COL0 -> MOSI
- K60 pad 1: COL0 -> MOSI
- K70 pad 1: COL0 -> MOSI
- U1 pad 18: unconnected-(U1-Pad18) -> COL8
- U1 pad 19: unconnected-(U1-Pad19) -> ROW1
- U1 pad 20: unconnected-(U1-Pad20) -> ROW2
- U1 pad 21: unconnected-(U1-Pad21) -> ROW6
- U1 pad 22: unconnected-(U1-Pad22) -> ROW7
- U1 pad 25: unconnected-(U1-Pad25) -> COL5
- U1 pad 26: unconnected-(U1-Pad26) -> COL6
- U1 pad 27: unconnected-(U1-Pad27) -> COL7
- U1 pad 28: unconnected-(U1-Pad28) -> ROW4
- U1 pad 29: unconnected-(U1-Pad29) -> ROW5
- U1 pad 36: unconnected-(U1-Pad36) -> COL4
- U1 pad 37: unconnected-(U1-Pad37) -> COL3
- U1 pad 38: unconnected-(U1-Pad38) -> COL2
- U1 pad 39: unconnected-(U1-Pad39) -> COL1
- U1 pad 40: unconnected-(U1-Pad40) -> ROW3
Routing:
- net MOSI: track 49.2 -> 496.5 mm, vias 1 -> 12
- net ROW2: track 0.00 -> 360.8 mm, vias 0 -> 14
- net ROW7: track 0.00 -> 342.8 mm, vias 0 -> 12
- net ROW6: track 0.00 -> 338.4 mm, vias 0 -> 10
- net ROW1: track 0.00 -> 322.5 mm, vias 0 -> 8
- net ROW3: track 0.00 -> 307.8 mm, vias 0 -> 6
- net ROW5: track 0.00 -> 301.9 mm, vias 0 -> 8
- net ROW4: track 0.00 -> 287.9 mm, vias 0 -> 8
- net COL1: track 221.6 -> 420.0 mm, vias 9 -> 13
- net COL2: track 239.9 -> 414.3 mm, vias 13 -> 17
- net COL0: track 145.6 -> 0.00 mm, vias 6 -> 0
- net COL3: track 310.5 -> 453.5 mm, vias 11 -> 15
- net COL4: track 342.6 -> 429.4 mm, vias 15 -> 19
- net COL5: track 185.8 -> 259.6 mm, vias 10 -> 13
- net Net-(DL10-Pad4): track 3.00 -> 65.1 mm, vias 0 -> 4
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- added copper zone on B.Cu, net GND
- added copper zone on F.Cu, net GND
Other:
- outline, holes or cut-outs redrawn

Commit message: PCB cleanup
Routing:
- net ROW4: track 287.9 -> 286.1 mm, vias 8 -> 6
- net COL1: track 420.0 -> 419.5 mm, vias 13 -> 11
- net COL2: track 414.3 -> 414.2 mm, vias 17 -> 15
- net COL3: vias 15 -> 13
- net GND: vias 19 -> 17

Commit message: Small PCB improvements
Parts:
- added JP2: HWB_EN, Jumper:SolderJumper-2_P1.3mm_Open_RoundedPad1.0x1.5mm, F.Cu at (120.9, 139.7)
Connections:
- net MOSI renamed COL0
- net SCK renamed ROW8
Routing:
- net Net-(SW2-Pad1): track 64.2 -> 72.0 mm, vias 4 -> 6
- net Net-(R2-Pad2): track 5.98 -> 9.24 mm
- net ROW7: track 342.8 -> 343.7 mm

Commit message: Initial fabrication files and update to Kailh socket parts
Changed lines of the file:
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@@
     (property "Sheetfile" "hedgehog-lite.kicad_sch")
     (property "Sheetname" "")
-    (attr exclude_from_pos_files)
+    (attr exclude_from_pos_files exclude_from_bom)
     (fp_text reference "JP1" (at 0 -1.8) (layer "F.SilkS")
       (effects (font (size 1 1) (thickness 0.15)))
@@
     (property "Sheetfile" "hedgehog-lite.kicad_sch")
     (property "Sheetname" "")
-    (attr through_hole exclude_from_pos_files)
+    (attr through_hole exclude_from_pos_files exclude_from_bom)
     (fp_text reference "J2" (at 0.635 -1.695) (layer "F.SilkS")
       (effects (font (size 1 1) (thickness 0.15)))
@@
     (fp_line (start -1 -0.625) (end 1 -0.625) (layer "F.Fab") (width 0.1))
     (fp_line (start 1 -0.625) (end 1 0.625) (layer "F.Fab") (width 0.1))
-    (pad "1" smd roundrect (at -0.9125 0 90) (size 1.025 1.4) (layers "F.Cu" "F.Paste" "F.Mask") (roundrect_rratio 0.243902)
+    (pad "1" smd roundrect (at -0.9125 0 90) (size 1.025 1.4) (layers "F.Cu" "F.Paste" "F.Mask") (roundrect_rratio 0.243902439)
       (net 118 "Net-(R4-Pad1)") (pintype "passive"))
-    (pad "2" smd roundrect (at 0.9125 0 90) (size 1.025 1.4) (layers "F.Cu" "F.Paste" "F.Mask") (roundrect_rratio 0.243902)
+    (pad "2" smd roundrect (at 0.9125 0 90) (size 1.025 1.4) (layers "F.Cu" "F.Paste" "F.Mask") (roundrect_rratio 0.243902439)
       (net 119 "DN") (pintype "passive"))
     (model "${KICAD6_3DMODEL_DIR}/Resistor_SMD.3dshapes/R_0805_2012Metric.wrl"
@@
     (property "Sheetfile" "hedgehog-lite.kicad_sch")
     (property "Sheetname" "")
-    (attr exclude_from_pos_files)
+    (attr exclude_from_pos_files exclude_from_bom)
     (fp_text reference "JP2" (at 0 -1.8) (layer "F.SilkS")
       (effects (font (size 1 1) (thickness 0.15)))
@@
     (fp_line (start -1 0.625) (end -1 -0.625) (layer "F.Fab") (width 0.1))
     (fp_line (start 1 0.625) (end -1 0.625) (layer "F.Fab") (width 0.1))
-    (pad "1" smd roundrect (at -0.9125 0) (size 1.025 1.4) (layers "F.Cu" "F.Paste" "F.Mask") (roundrect_rratio 0.243902)
+    (pad "1" smd roundrect (at -0.9125 0) (size 1.025 1.4) (layers "F.Cu" "F.Paste" "F.Mask") (roundrect_rratio 0.243902439)
       (net 3 "GND") (pintype "passive"))
-    (pad "2" smd roundrect (at 0.9125 0) (size 1.025 1.4) (layers "F.Cu" "F.Paste" "F.Mask") (roundrect_rratio 0.243902)
+    (pad "2" smd roundrect (at 0.9125 0) (size 1.025 1.4) (layers "F.Cu" "F.Paste" "F.Mask") (roundrect_rratio 0.243902439)
       (net 13 "Net-(R2-Pad2)") (pintype "passive"))
     (model "${KICAD6_3DMODEL_DIR}/Resistor_SMD.3dshapes/R_0805_2012Metric.wrl"
@@
     (fp_line (start -1 0.625) (end -1 -0.625) (layer "F.Fab") (width 0.1))
     (fp_line (start -1 -0.625) (end 1 -0.625) (layer "F.Fab") (width 0.1))
-    (pad "1" smd roundrect (at -0.9125 0 90) (size 1.025 1.4) (layers "F.Cu" "F.Paste" "F.Mask") (roundrect_rratio 0.243902)
+    (pad "1" smd roundrect (at -0.9125 0 90) (size 1.025 1.4) (layers "F.Cu" "F.Paste" "F.Mask") (roundrect_rratio 0.243902439)
       (net 117 "Net-(R3-Pad1)") (pintype "passive"))
-    (pad "2" smd roundrect (at 0.9125 0 90) (size 1.025 1.4) (layers "F.Cu" "F.Paste" "F.Mask") (roundrect_rratio 0.243902)
+    (pad "2" smd roundrect (at 0.9125 0 90) (size 1.025 1.4) (layers "F.Cu" "F.Paste" "F.Mask") (roundrect_rratio 0.243902439)
       (net 120 "DP") (pintype "passive"))
     (model "${KICAD6_3DMODEL_DIR}/Resistor_SMD.3dshapes/R_0805_2012Metric.wrl"
@@
     (property "Sheetfile" "hedgehog-lite.kicad_sch")
     (property "Sheetname" "")
-    (attr smd exclude_from_pos_files)
+    (attr smd exclude_from_pos_files exclude_from_bom)
     (fp_text reference "SW1" (at 0 3.75) (layer "B.SilkS")
       (effects (font (size 1 1) (thickness 0.15)) (justify mirror))

Commit message: Added logos CR
Other:
- board text added: "Hedgehog Lite 60"
- board text added: "v 1.0 © git: max3-2"
